Commit message: added moveit2 config package

File: omron1s_urdf/urdf/omron1s.xacro (robot description, xacro)
@@ -49,5 +49,6 @@
     </inertial>
   </link>
-  <joint name="joint1" type="continuous">
+  <joint name="joint1" type="revolute">
+    <limit lower="-6.28" upper="6.28" effort="100" velocity="6.28"/>
     <parent link="link1"/>
     <child link="link2"/>
@@ -77,5 +78,6 @@
     </inertial>
   </link>
-  <joint name="joint2" type="continuous">
+  <joint name="joint2" type="revolute">
+    <limit lower="-6.28" upper="6.28" effort="100" velocity="6.28"/>
     <parent link="link2"/>
     <child link="link3"/>

Commit message: fix srdf for ee

File: omron1s_urdf/urdf/omron1s.xacro (robot description, xacro)
@@ -50,5 +50,5 @@
   </link>
   <joint name="joint1" type="revolute">
-    <limit lower="-6.28" upper="6.28" effort="100" velocity="6.28"/>
+    <limit lower="-3.14" upper="3.14" effort="100" velocity="6.28"/>
     <parent link="link1"/>
     <child link="link2"/>
@@ -79,5 +79,5 @@
   </link>
   <joint name="joint2" type="revolute">
-    <limit lower="-6.28" upper="6.28" effort="100" velocity="6.28"/>
+    <limit lower="-3.14" upper="3.14" effort="100" velocity="6.28"/>
     <parent link="link2"/>
     <child link="link3"/>
