Commit message: simulation with gazebo

File: omron1s_description/urdf/omron1s.xacro (robot description, xacro)
@@ -34,5 +34,5 @@
       <geometry>
         <mesh
-          filename="package://omron1s_description/meshes/base_link.STL" />
+          filename="file:///$(find omron1s_description)/meshes/base_link.STL" />
       </geometry>
       <material
@@ -48,5 +48,5 @@
       <geometry>
         <mesh
-          filename="package://omron1s_description/meshes/base_link.STL" />
+          filename="file:///$(find omron1s_description)/meshes/base_link.STL" />
       </geometry>
     </collision>
@@ -74,5 +74,5 @@
       <geometry>
         <mesh
-          filename="package://omron1s_description/meshes/link1.STL" />
+          filename="file:///$(find omron1s_description)/meshes/link1.STL" />
       </geometry>
       <material
@@ -88,5 +88,5 @@
       <geometry>
         <mesh
-          filename="package://omron1s_description/meshes/link1.STL" />
+          filename="file:///$(find omron1s_description)/meshes/link1.STL" />
       </geometry>
     </collision>
@@ -107,6 +107,7 @@
       lower="-3.14"
       upper="3.14"
-      effort="100"
+      effort="500"
       velocity="6.28" />
+    <dynamics damping="60.0" friction="4.0" />
   </joint>
   <link
@@ -132,5 +133,5 @@
       <geometry>
         <mesh
-          filename="package://omron1s_description/meshes/link2.STL" />
+          filename="file:///$(find omron1s_description)/meshes/link2.STL" />
       </geometry>
       <material
@@ -146,5 +147,5 @@
       <geometry>
         <mesh
-          filename="package://omron1s_description/meshes/link2.STL" />
+          filename="file:///$(find omron1s_description)/meshes/link2.STL" />
       </geometry>
     </collision>
@@ -165,6 +166,7 @@
       lower="-3.14"
       upper="3.14"
-      effort="100"
+      effort="500"
       velocity="6.28" />
+    <dynamics damping="60.0" friction="4.0" />
   </joint>
   <link
@@ -190,5 +192,5 @@
       <geometry>
         <mesh
-          filename="package://omron1s_description/meshes/link3.STL" />
+          filename="file:///$(find omron1s_description)/meshes/link3.STL" />
       </geometry>
       <material
@@ -204,5 +206,5 @@
       <geometry>
         <mesh
-          filename="package://omron1s_description/meshes/link3.STL" />
+          filename="file:///$(find omron1s_description)/meshes/link3.STL" />
       </geometry>
     </collision>
@@ -223,6 +225,7 @@
       lower="-3.14"
       upper="3.14"
-      effort="100"
+      effort="500"
       velocity="6.28" />
+    <dynamics damping="60.0" friction="4.0" />
   </joint>
   <link
@@ -248,5 +251,5 @@
       <geometry>
         <mesh
-          filename="package://omron1s_description/meshes/link4.STL" />
+          filename="file:///$(find omron1s_description)/meshes/link4.STL" />
       </geometry>
       <material
@@ -262,5 +265,5 @@
       <geometry>
         <mesh
-          filename="package://omron1s_description/meshes/link4.STL" />
+          filename="file:///$(find omron1s_description)/meshes/link4.STL" />
       </geometry>
     </collision>
@@ -281,8 +284,10 @@
       lower="-3.14"
       upper="3.14"
-      effort="100"
+      effort="500"
       velocity="6.28" />
+    <dynamics damping="60.0" friction="4.0" />
   </joint>
-    <ros2_control name="Omron1SHardware" type="system">
+    <!-- ROS2 CONTROL REAL -->
+    <!-- <ros2_control name="Omron1SHardware" type="system">
       <hardware>
         <plugin>omron1s_hardware/Omron1SHardware</plugin>
@@ -310,4 +315,98 @@
         <state_interface name="position"/>
       </joint>
-    </ros2_control>
+    </ros2_control> -->
+    <!-- ROS2 CONTROL SIMULATION -->
+    <ros2_control name="GazeboSystem" type="system">
+			<hardware>
+				<plugin>gazebo_ros2_control/GazeboSystem</plugin>
+	    </hardware>
+	    	<joint name="joint1">
+	    		<command_interface name="position">
+	    			<param name="min">-3.14</param>
+	    			<param name="max">3.14</param>
+	    		</command_interface>
+	    		<state_interface name="position"/>
+	    		<state_interface name="velocity"/>
+	    		<state_interface name="effort"/>
+	    	</joint>
+	    	<joint name="joint2">
+	    		<command_interface name="position">
+	    			<param name="min">-3.14</param>
+	    			<param name="max">3.14</param>
+	    		</command_interface>
+	    		<state_interface name="position"/>
+	    		<state_interface name="velocity"/>
+	    		<state_interface name="effort"/>
+	    	</joint>
+	    	<joint name="joint3">
+	    		<command_interface name="position">
+	    			<param name="min">-3.14</param>
+	    			<param name="max">3.14</param>
+	    		</command_interface>
+	    		<state_interface name="position"/>
+	    		<state_interface name="velocity"/>
+	    		<state_interface name="effort"/>
+	    	</joint>
+	    	<joint name="joint4">
+	    		<command_interface name="position">
+	    			<param name="min">-3.14</param>
+	    			<param name="max">3.14</param>
+	    		</command_interface>
+	    		<state_interface name="position"/>
+	    		<state_interface name="velocity"/>
+	    		<state_interface name="effort"/>
+	    	</joint>
+	  	</ros2_control>
+		<gazebo>
+			<plugin name="gazebo_ros2_control" filename="libgazebo_ros2_control.so">
+        		<!--<robot_sim_type>gazebo_ros2_control/DefaultRobotHWSim</robot_sim_type> -->
+				<!-- <robot_sim_type>gazebo_ros2_control/GazeboSystem</robot_sim_type> -->
+				<parameters>$(find omron1s_hwi)/config/controller_configuration.yaml</parameters>
+		  </plugin>
+		</gazebo>
+    <!-- TRANSMISSION -->
+    <!-- Transmission 1 -->
+		<transmission name="tran1">
+			<type>transmission_interface/SimpleTransmission</type>
+			<joint name="joint1">
+				<hardwareInterface>hardware_interface/PositionJointInterface</hardwareInterface>
+			</joint>
+			<actuator name="motor1">
+				<hardwareInterface>hardware_interface/PositionJointInterface</hardwareInterface>
+				<mechanicalReduction>1</mechanicalReduction>
+			</actuator>
+		</transmission>
+		<!-- Transmission 2 -->
+		<transmission name="tran2">
+			<type>transmission_interface/SimpleTransmission</type>
+			<joint name="joint2">
+				<hardwareInterface>hardware_interface/PositionJointInterface</hardwareInterface>
+			</joint>
+			<actuator name="motor2">
+				<hardwareInterface>hardware_interface/PositionJointInterface</hardwareInterface>
+				<mechanicalReduction>1</mechanicalReduction>
+			</actuator>
+		</transmission>
+		<!-- Transmission 3 -->
+		<transmission name="tran3">
+			<type>transmission_interface/SimpleTransmission</type>
+			<joint name="joint3">
+				<hardwareInterface>hardware_interface/PositionJointInterface</hardwareInterface>
+			</joint>
+			<actuator name="motor3">
+				<hardwareInterface>hardware_interface/PositionJointInterface</hardwareInterface>
+				<mechanicalReduction>1</mechanicalReduction>
+			</actuator>
+		</transmission>
+		<!-- Transmission 4 -->
+		<transmission name="tran4">
+			<type>transmission_interface/SimpleTransmission</type>
+			<joint name="joint4">
+				<hardwareInterface>hardware_interface/PositionJointInterface</hardwareInterface>
+			</joint>
+			<actuator name="motor4">
+				<hardwareInterface>hardware_interface/PositionJointInterface</hardwareInterface>
+				<mechanicalReduction>1</mechanicalReduction>
+			</actuator>
+		</transmission>
 </robot>

Commit message: update ros2_control tag in xacro

File: omron1s_description/urdf/omron1s.xacro (robot description, xacro)
@@ -288,38 +288,16 @@
     <dynamics damping="60.0" friction="4.0" />
   </joint>
-    <!-- ROS2 CONTROL REAL -->
-    <!-- <ros2_control name="Omron1SHardware" type="system">
-      <hardware>
+    <!-- ROS2 CONTROL-->
+    <ros2_control name="Omron1SControl" type="system">
+      <!-- <hardware>
         <plugin>omron1s_hardware/Omron1SHardware</plugin>
         <param name="interface_name">enp2s0</param>
         <param name="use_dummy">false</param>
-      </hardware>
-      <joint name="joint1">
-        <param name="id">1</param>
-        <command_interface name="position"/>
-        <state_interface name="position"/>
-      </joint>
-      <joint name="joint2">
-        <param name="id">2</param>
-        <command_interface name="position"/>
-        <state_interface name="position"/>
-      </joint>
-      <joint name="joint3">
-        <param name="id">3</param>
-        <command_interface name="position"/>
-        <state_interface name="position"/>
-      </joint>
-      <joint name="joint4">
-        <param name="id">4</param>
-        <command_interface name="position"/>
-        <state_interface name="position"/>
-      </joint>
-    </ros2_control> -->
-    <!-- ROS2 CONTROL SIMULATION -->
-    <ros2_control name="GazeboSystem" type="system">
+      </hardware> -->
 			<hardware>
 				<plugin>gazebo_ros2_control/GazeboSystem</plugin>
 	    </hardware>
 	    	<joint name="joint1">
+          <param name="id">1</param>
 	    		<command_interface name="position">
 	    			<param name="min">-3.14</param>
@@ -331,4 +309,5 @@
 	    	</joint>
 	    	<joint name="joint2">
+          <param name="id">2</param>
 	    		<command_interface name="position">
 	    			<param name="min">-3.14</param>
@@ -340,4 +319,5 @@
 	    	</joint>
 	    	<joint name="joint3">
+          <param name="id">3</param>
 	    		<command_interface name="position">
 	    			<param name="min">-3.14</param>
@@ -349,4 +329,5 @@
 	    	</joint>
 	    	<joint name="joint4">
+          <param name="id">4</param>
 	    		<command_interface name="position">
 	    			<param name="min">-3.14</param>

Commit message: update omron1s_description

File: omron1s_description/urdf/omron1s.xacro (robot description, xacro)
@@ -16,5 +16,5 @@
     <inertial>
       <origin
-        xyz="0.058756 -0.084662 0.1005"
+        xyz="0.058756 0.1005 0.084662"
         rpy="0 0 0" />
       <mass
@@ -22,9 +22,9 @@
       <inertia
         ixx="0.0032491"
-        ixy="-2.2578E-22"
-        ixz="9.8868E-22"
-        iyy="0.0032491"
-        iyz="-6.6907E-19"
-        izz="0.0048171" />
+        ixy="1.0152E-21"
+        ixz="2.3749E-22"
+        iyy="0.0048171"
+        iyz="7.6509E-19"
+        izz="0.0032491" />
     </inertial>
     <visual>
@@ -56,15 +56,15 @@
     <inertial>
       <origin
-        xyz="2.08166817117217E-17 0.04 -0.0377780415986943"
-        rpy="0 0 0" />
-      <mass
-        value="2.08761053730566" />
-      <inertia
-        ixx="0.00742870445718791"
-        ixy="-6.84015806136404E-20"
-        ixz="1.95156391047391E-18"
-        iyy="0.00952055836647544"
-        iyz="1.02543660202385E-19"
-        izz="0.00422480958182635" />
+        xyz="-2.7756E-17 0.04 -0.037778"
+        rpy="0 0 0" />
+      <mass
+        value="2.0876" />
+      <inertia
+        ixx="0.0074287"
+        ixy="-4.9804E-20"
+        ixz="-4.391E-18"
+        iyy="0.0095206"
+        iyz="1.2084E-19"
+        izz="0.0042248" />
     </inertial>
     <visual>
@@ -79,5 +79,5 @@
         name="">
         <color
-          rgba="0.792156862745098 0.819607843137255 0.933333333333333 1" />
+          rgba="0.79216 0.81961 0.93333 1" />
       </material>
     </visual>
@@ -96,6 +96,6 @@
     type="revolute">
     <origin
-      xyz="0.0587564520357434 -0.0846616099911215 0.151979361094108"
-      rpy="1.5707963267949 0 -2.77072298333055" />
+      xyz="0.058756 -0.084662 0.15198"
+      rpy="1.5708 0 -2.9046" />
     <parent
       link="base_link" />
@@ -105,9 +105,11 @@
       xyz="0 1 0" />
     <limit
-      lower="-3.14"
-      upper="3.14"
+      lower="-6.28"
+      upper="6.28"
       effort="500"
       velocity="6.28" />
-    <dynamics damping="60.0" friction="4.0" />
+    <dynamics
+      damping="200"
+      friction="50" />
   </joint>
   <link
@@ -115,15 +117,15 @@
     <inertial>
       <origin
-        xyz="-0.095000000000001 -2.77555756156289E-16 0.275"
-        rpy="0 0 0" />
-      <mass
-        value="2.45132741228718" />
-      <inertia
-        ixx="0.0781860308173814"
-        ixy="0"
-        ixz="4.32325616278595E-18"
-        iyy="0.0774228597300263"
-        iyz="7.23162849047831E-17"
-        izz="0.00178455750914138" />
+        xyz="-0.022244 -3.8858E-16 0.275"
+        rpy="0 0 0" />
+      <mass
+        value="2.4513" />
+      <inertia
+        ixx="0.078186"
+        ixy="-1.7347E-18"
+        ixz="-3.5521E-17"
+        iyy="0.077423"
+        iyz="1.0148E-16"
+        izz="0.0017846" />
     </inertial>
     <visual>
@@ -138,5 +140,5 @@
         name="">
         <color
-          rgba="0.792156862745098 0.819607843137255 0.933333333333333 1" />
+          rgba="0.79216 0.81961 0.93333 1" />
       </material>
     </visual>
@@ -155,6 +157,6 @@
     type="revolute">
     <origin
-      xyz="0 0.0400000000000031 -0.0999999999999985"
-      rpy="1.97667516838365 0 3.14159265358979" />
+      xyz="0.072756 0.04 -0.1"
+      rpy="1.1256 0 3.1416" />
     <parent
       link="link1" />
@@ -164,9 +166,11 @@
       xyz="1 0 0" />
     <limit
-      lower="-3.14"
-      upper="3.14"
+      lower="-6.28"
+      upper="6.28"
       effort="500"
       velocity="6.28" />
-    <dynamics damping="60.0" friction="4.0" />
+    <dynamics
+      damping="200"
+      friction="50" />
   </joint>
   <link
@@ -174,15 +178,15 @@
     <inertial>
       <origin
-        xyz="-0.0449999999999999 -2.22044604925031E-16 0.275"
-        rpy="0 0 0" />
-      <mass
-        value="2.45132741228718" />
-      <inertia
-        ixx="0.0781860308173814"
-        ixy="-4.33680868994202E-18"
-        ixz="6.39679281766448E-18"
-        iyy="0.0774228597300263"
-        iyz="9.83371370444353E-17"
-        izz="0.00178455750914137" />
+        xyz="0.027756 8.8818E-16 0.275"
+        rpy="0 0 0" />
+      <mass
+        value="2.4513" />
+      <inertia
+        ixx="0.078186"
+        ixy="-4.3368E-19"
+        ixz="-2.1467E-17"
+        iyy="0.077423"
+        iyz="5.9902E-17"
+        izz="0.0017846" />
     </inertial>
     <visual>
@@ -197,5 +201,5 @@
         name="">
         <color
-          rgba="0.792156862745098 0.819607843137255 0.933333333333333 1" />
+          rgba="0.79216 0.81961 0.93333 1" />
       </material>
     </visual>
@@ -215,5 +219,5 @@
     <origin
       xyz="0 0 0.55"
-      rpy="1.75653072975658 0 0" />
+      rpy="2.4678 0 0" />
     <parent
       link="link2" />
@@ -223,9 +227,11 @@
       xyz="1 0 0" />
     <limit
-      lower="-3.14"
-      upper="3.14"
+      lower="-6.28"
+      upper="6.28"
       effort="500"
       velocity="6.28" />
-    <dynamics damping="60.0" friction="4.0" />
+    <dynamics
+      damping="200"
+      friction="50" />
   </joint>
   <link
@@ -233,15 +239,15 @@
     <inertial>
       <origin
-        xyz="-0.048723 -1.4225E-08 2.0409E-08"
-        rpy="0 0 0" />
-      <mass
-        value="0.95838" />
-      <inertia
-        ixx="0.00129"
-        ixy="8.6782E-10"
-        ixz="-2.1532E-09"
-        iyy="0.0016328"
-        iyz="-9.2513E-10"
-        izz="0.0017839" />
+        xyz="0.01137 -1.4733E-08 2.4175E-08"
+        rpy="0 0 0" />
+      <mass
+        value="0.95052" />
+      <inertia
+        ixx="0.001281"
+        ixy="8.7095E-10"
+        ixz="-2.2716E-09"
+        iyy="0.0016268"
+        iyz="-9.4098E-10"
+        izz="0.0017739" />
     </inertial>
     <visual>
@@ -273,6 +279,6 @@
     type="revolute">
     <origin
-      xyz="0 0 0.55"
-      rpy="0.535953139821402 0 -3.14159265358979" />
+      xyz="0.13276 0 0.55"
+      rpy="0.45181 0 -3.1416" />
     <parent
       link="link3" />
@@ -280,114 +286,169 @@
       link="link4" />
     <axis
-      xyz="1 0 0" />
+      xyz="-1 0 0" />
     <limit
-      lower="-3.14"
-      upper="3.14"
+      lower="-6.28"
+      upper="6.28"
       effort="500"
       velocity="6.28" />
-    <dynamics damping="60.0" friction="4.0" />
-  </joint>
-    <!-- ROS2 CONTROL-->
-    <ros2_control name="Omron1SControl" type="system">
-      <!-- <hardware>
-        <plugin>omron1s_hardware/Omron1SHardware</plugin>
-        <param name="interface_name">enp2s0</param>
-        <param name="use_dummy">false</param>
-      </hardware> -->
-			<hardware>
-				<plugin>gazebo_ros2_control/GazeboSystem</plugin>
-	    </hardware>
-	    	<joint name="joint1">
-          <param name="id">1</param>
-	    		<command_interface name="position">
-	    			<param name="min">-3.14</param>
-	    			<param name="max">3.14</param>
-	    		</command_interface>
-	    		<state_interface name="position"/>
-	    		<state_interface name="velocity"/>
-	    		<state_interface name="effort"/>
-	    	</joint>
-	    	<joint name="joint2">
-          <param name="id">2</param>
-	    		<command_interface name="position">
-	    			<param name="min">-3.14</param>
-	    			<param name="max">3.14</param>
-	    		</command_interface>
-	    		<state_interface name="position"/>
-	    		<state_interface name="velocity"/>
-	    		<state_interface name="effort"/>
-	    	</joint>
-	    	<joint name="joint3">
-          <param name="id">3</param>
-	    		<command_interface name="position">
-	    			<param name="min">-3.14</param>
-	    			<param name="max">3.14</param>
-	    		</command_interface>
-	    		<state_interface name="position"/>
-	    		<state_interface name="velocity"/>
-	    		<state_interface name="effort"/>
-	    	</joint>
-	    	<joint name="joint4">
-          <param name="id">4</param>
-	    		<command_interface name="position">
-	    			<param name="min">-3.14</param>
-	    			<param name="max">3.14</param>
-	    		</command_interface>
-	    		<state_interface name="position"/>
-	    		<state_interface name="velocity"/>
-	    		<state_interface name="effort"/>
-	    	</joint>
-	  	</ros2_control>
-		<gazebo>
-			<plugin name="gazebo_ros2_control" filename="libgazebo_ros2_control.so">
-        		<!--<robot_sim_type>gazebo_ros2_control/DefaultRobotHWSim</robot_sim_type> -->
-				<!-- <robot_sim_type>gazebo_ros2_control/GazeboSystem</robot_sim_type> -->
-				<parameters>$(find omron1s_hwi)/config/controller_configuration.yaml</parameters>
-		  </plugin>
-		</gazebo>
-    <!-- TRANSMISSION -->
-    <!-- Transmission 1 -->
-		<transmission name="tran1">
-			<type>transmission_interface/SimpleTransmission</type>
-			<joint name="joint1">
-				<hardwareInterface>hardware_interface/PositionJointInterface</hardwareInterface>
-			</joint>
-			<actuator name="motor1">
-				<hardwareInterface>hardware_interface/PositionJointInterface</hardwareInterface>
-				<mechanicalReduction>1</mechanicalReduction>
-			</actuator>
-		</transmission>
-		<!-- Transmission 2 -->
-		<transmission name="tran2">
-			<type>transmission_interface/SimpleTransmission</type>
-			<joint name="joint2">
-				<hardwareInterface>hardware_interface/PositionJointInterface</hardwareInterface>
-			</joint>
-			<actuator name="motor2">
-				<hardwareInterface>hardware_interface/PositionJointInterface</hardwareInterface>
-				<mechanicalReduction>1</mechanicalReduction>
-			</actuator>
-		</transmission>
-		<!-- Transmission 3 -->
-		<transmission name="tran3">
-			<type>transmission_interface/SimpleTransmission</type>
-			<joint name="joint3">
-				<hardwareInterface>hardware_interface/PositionJointInterface</hardwareInterface>
-			</joint>
-			<actuator name="motor3">
-				<hardwareInterface>hardware_interface/PositionJointInterface</hardwareInterface>
-				<mechanicalReduction>1</mechanicalReduction>
-			</actuator>
-		</transmission>
-		<!-- Transmission 4 -->
-		<transmission name="tran4">
-			<type>transmission_interface/SimpleTransmission</type>
-			<joint name="joint4">
-				<hardwareInterface>hardware_interface/PositionJointInterface</hardwareInterface>
-			</joint>
-			<actuator name="motor4">
-				<hardwareInterface>hardware_interface/PositionJointInterface</hardwareInterface>
-				<mechanicalReduction>1</mechanicalReduction>
-			</actuator>
-		</transmission>
+    <dynamics
+      damping="200"
+      friction="50" />
+  </joint>
+  <link
+    name="gripper">
+    <inertial>
+      <origin
+        xyz="0.037654 0.05165 0.064091"
+        rpy="0 0 0" />
+      <mass
+        value="0.25674" />
+      <inertia
+        ixx="0.00015569"
+        ixy="1.8365E-07"
+        ixz="2.3502E-07"
+        iyy="0.00027921"
+        iyz="9.4751E-08"
+        izz="0.00021782" />
+    </inertial>
+    <visual>
+      <origin
+        xyz="0 0 0"
+        rpy="0 0 0" />
+      <geometry>
+        <mesh
+          filename="file:///$(find omron1s_description)/meshes/gripper.STL" />
+      </geometry>
+      <material
+        name="">
+        <color
+          rgba="0.75294 0.75294 0.75294 1" />
+      </material>
+    </visual>
+    <collision>
+      <origin
+        xyz="0 0 0"
+        rpy="0 0 0" />
+      <geometry>
+        <mesh
+          filename="file:///$(find omron1s_description)/meshes/gripper.STL" />
+      </geometry>
+    </collision>
+  </link>
+  <joint
+    name="gripper_joint"
+    type="fixed">
+    <origin
+      xyz="0.037522 0.15383 -0.064188"
+      rpy="0 0 3.1416" />
+    <parent
+      link="link4" />
+    <child
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
Commit message: kinematics test

File: omron1s_description/urdf/omron1s.xacro (robot description, xacro)
@@ -346,4 +346,18 @@
     <child
       link="gripper" />
+    <axis
+      xyz="0 0 0" />
+  </joint>
+  <link name="gripper_tip"/>
+  <joint
+    name="gripper_tip_joint"
+    type="fixed">
+    <origin
+      xyz="0.0 0.0 0.0"
+      rpy="0 0 0" />
+    <parent
+      link="gripper" />
+    <child
+      link="gripper_tip" />
     <axis
       xyz="0 0 0" />
