Commit message: +

File: omron1s_description/urdf/omron1s.xacro (robot description, xacro)
@@ -8,13 +8,35 @@
   <!-- Used for fixing robot to Gazebo 'base_link' -->
   <link name="world"/>
-  <joint name="fixed" type="fixed">
+  <!-- <joint name="fixed" type="fixed">
     <parent link="world"/>
     <child link="base_link"/>
-  </joint>
+  </joint> -->
+    <joint
+    name="fixed"
+    type="fixed">
+    <origin
+      xyz="-0.097 -0.037 0.0"
+      rpy="0 0 1.3326126" />
+    <parent
+      link="world" />
+    <child
+      link="base_link" />
+  </joint>
+    <!-- <joint
+    name="fixed"
+    type="fixed">
+    <origin
+      xyz="0.059 -0.085 0.052"
+      rpy="0 0 -1.3326126" />
+    <parent
+      link="world" />
+    <child
+      link="base_link" />
+  </joint> -->
   <link
     name="base_link">
     <inertial>
       <origin
-        xyz="0.058756 0.1005 0.084662"
+        xyz="0 0 0"
         rpy="0 0 0" />
       <mass
@@ -349,18 +371,28 @@
       xyz="0 0 0" />
   </joint>
-  <link name="gripper_tip"/>
-  <joint
-    name="gripper_tip_joint"
+  <link name="tool0"/>
+  <joint
+    name="tool0_joint"
     type="fixed">
     <origin
-      xyz="0.0 0.0 0.0"
-      rpy="0 0 0" />
-    <parent
-      link="gripper" />
-    <child
-      link="gripper_tip" />
-    <axis
-      xyz="0 0 0" />
-  </joint>
+      xyz="0.0 0.19 0.0"
+      rpy="1.5708 -1.5708 0" />
+    <parent
+      link="link4" />
+    <child
+      link="tool0" />
+  </joint>
+  <!-- <link name="poseref"/>
+  <joint
+    name="poseref_joint"
+    type="fixed">
+    <origin
+      xyz="0.059 -0.085 0.052"
+      rpy="0 0 -1.3326126" />
+    <parent
+      link="base_link" />
+    <child
+      link="poseref" />
+  </joint> -->
   <!-- ROS2 CONTROL-->
   <ros2_control name="Omron1SControl" type="system">
